File: car-instrument-panel.kicad_sch (KiCad schematic)
At the start: 27 parts, among them J1 Conn_01x03, Q1 2N3904, Q2 2N3904, Q3 2N3904, Q4 2N3904, Q5 2N3904, U1 LM1602A, U2 RaspberryPi-Pico, U3 74HC595, U4 HS420561K-32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

Commit message: old changes
Connections:
- net TACHOMETER: no longer U2.2 (GPIO1)
Other:
- note added: "TODO: Add level shifter"
- note removed: "Might need to connect RCLK to a different GPIO. Possible that CS can be configured to trigger latch."
Changed lines of the file:
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@@
-    (stroke (width 0) (type default) (color 0 0 0 0))
-  )
-  (wire (pts (xy 167.64 95.25) (xy 167.64 88.9))
     (stroke (width 0) (type default) (color 0 0 0 0))
   )
@@
     (stroke (width 0) (type default) (color 0 0 0 0))
   )
+  (text "TODO:\nAdd level shifter" (at 162.56 93.98 0)
+    (effects (font (size 1.27 1.27)) (justify left bottom))
+  )
   (text "typical VDD-V0=4.5V\nV0=0.5V\npot set to ~10%" (at 167.64 130.81 180)
     (effects (font (size 1.27 1.27)) (justify right bottom))
@@
     (effects (font (size 1.27 1.27)) (justify right bottom))
   )
-  (text "Might need to connect RCLK to \na different GPIO. Possible that \nCS can be configured to trigger\nlatch."
-    (at 88.9 52.07 0)
-    (effects (font (size 1.27 1.27)) (justify left bottom))
-  )
   (label "SEG2" (at 172.72 44.45 0)
